Commit message: Added inertia to simple robot urdf and added the example urdf from notion

File: urdf/simple_rover.urdf (robot description, URDF)
Before this commit: robot simple_rover, 5 links, 4 joints
Links:
- link back_left_wheel: mass None -> 0.5
- link back_right_wheel: mass None -> 0.5
- link base_link: mass None -> 0.5
- link front_left_wheel: mass None -> 0.5; geometry collision cylinder length=0.04 radius=0.1; visual cylinder length=0.04 radius=0.1
- link front_right_wheel: mass None -> 0.5

Commit message: updated simple_rover.urdf

File: urdf/simple_rover.urdf (robot description, URDF)
Before this commit: robot simple_rover, 5 links, 4 joints
Links:
- link base_link: mass 0.5 -> 5.0

Commit message: SPAWNING ROVER NOW WOOOOO

File: urdf/simple_rover.urdf (robot description, URDF)
Before this commit: robot simple_rover, 5 links, 4 joints
Joints:
- joint back_left_wheel_joint: limit (none) -> effort=10000 velocity=1000
- joint back_right_wheel_joint: limit (none) -> effort=10000 velocity=1000
- joint front_left_wheel_joint: limit (none) -> effort=10000 velocity=1000
- joint front_right_wheel_joint: limit (none) -> effort=10000 velocity=1000
