Commit message: Set up differential drive in URDF

File: urdf/rover.urdf (robot description, URDF)
Before this commit: robot URDF Model, 7 links, 6 joints
Links:
- removed link Front Left Wheel
- removed link Front Right Wheel
- removed link Rear Left Wheel
- removed link Rear Right Wheel
- added link front_left_wheel, mass 2.5634; collision mesh filename=package://simple_robot_description/meshes/Front_Left_Wheel.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; visual mesh filename=package://simple_robot_description/meshes/Front_Left_Wheel.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
- added link front_right_wheel, mass 2.5634; collision mesh filename=package://simple_robot_description/meshes/Front_Right_Wheel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; visual mesh filename=package://simple_robot_description/meshes/Front_Right_Wheel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
- added link rear_left_wheel, mass 2.5634; collision mesh filename=package://simple_robot_description/meshes/Rear_Left_Wheel.s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; visual mesh filename=package://simple_robot_description/meshes/Rear_Left_Wheel.s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
- added link rear_right_wheel, mass 2.5634; collision mesh filename=package://simple_robot_description/meshes/Rear_Right_Wheel.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; visual mesh filename=package://simple_robot_description/meshes/Rear_Right_Wheel.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
Joints:
- removed joint Front Left Wheel Joint
- removed joint Front Right Wheel Joint
- removed joint Rear Left Wheel Joint
- removed joint Rear Right Wheel Joint
- added joint front_left_wheel_joint: type continuous, parent Left Rocker, child front_left_wheel, origin xyz=0.065325 -0.17676 0.2723 rpy=0 0 1.5708, axis 0 1 0, limit effort=5 velocity=10
- added joint front_right_wheel_joint: type continuous, parent Right Rocker, child front_right_wheel, origin xyz=-0.065325 -0.18923 0.26378 rpy=0 0.019168 -1.5708, axis 0 1 0, limit effort=5 velocity=10
- added joint rear_left_wheel_joint: type continuous, parent Left Rocker, child rear_left_wheel, origin xyz=0.065325 -0.19309 -0.26097 rpy=0 0.025218 1.5708, axis 0 1 0, limit effort=5 velocity=10
- added joint rear_right_wheel_joint: type continuous, parent Right Rocker, child rear_right_wheel, origin xyz=-0.065325 -0.18074 -0.26967 rpy=0 0.019168 -1.5708, axis 0 1 0, limit effort=5 velocity=10

Commit message: Rover now turns and drives with 4 wheels

File: urdf/rover.urdf (robot description, URDF)
Before this commit: robot URDF Model, 7 links, 6 joints
Joints:
- joint front_left_wheel_joint: axis 0 1 0 -> 0 -1 0
- joint rear_left_wheel_joint: axis 0 1 0 -> 0 -1 0

File: urdf/simple_rover.urdf (robot description, URDF)
Before this commit: robot simple_rover, 5 links, 4 joints
Joints:
- joint back_right_wheel_joint: axis 0 1 0 -> 0 -1 0
- joint front_right_wheel_joint: axis 0 1 0 -> 0 -1 0
